Commit message: syntax clean up: +joint limits

File: arctos_urdf_description/urdf/arctos_urdf.urdf (robot description, URDF)
Before this commit: robot arctos_urdf, 0 links, 9 joints
Joints:
- removed joint gripper
- removed joint jaw1
- removed joint jaw2
- removed joint joint1
- removed joint joint2
- removed joint joint3
- removed joint joint4
- removed joint joint5
- removed joint joint6

File: arctos_urdf_description/urdf/joint_link.xacro (robot description, xacro)
@@ -1,9 +1,6 @@
 <?xml version="1.0"?>
 <robot xmlns:xacro="http://www.ros.org/wiki/xacro" name="arctos_urdf">
-<xacro:macro name="arctos_link" params="name origin_xyz origin_rpy material_name">
+<xacro:macro name="arctos_link" params="name origin_xyz origin_rpy material_name inertia_origin_xyz inertia_origin_rpy mass ixx iyy izz ixy iyz ixz">
   <link name="${name}">
-    <inertial>
-      <xacro:insert_block name="inertial_properties"/>
-    </inertial>
     <visual>
       <origin xyz="${origin_xyz}" rpy="${origin_rpy}"/>
@@ -19,4 +16,9 @@
       </geometry>
     </collision>
+    <inertial>
+      <origin xyz="${inertia_origin_xyz}" rpy="${inertia_origin_rpy}"/>
+      <mass value="${mass}"/>
+      <inertia ixx="${ixx}" iyy="${iyy}" izz="${izz}" ixy="${ixy}" iyz="${iyz}" ixz="${ixz}"/>
+    </inertial>
   </link>
 </xacro:macro>
@@ -30,3 +32,15 @@
   </joint>
 </xacro:macro>
+<xacro:macro name="transmission" params="name joint_name actuator_name">
+  <transmission name="${name}">
+    <type>transmission_interface/SimpleTransmission</type>
+    <joint name="${joint_name}">
+      <hardwareInterface>hardware_interface/EffortJointInterface</hardwareInterface>
+    </joint>
+    <actuator name="${actuator_name}">
+      <hardwareInterface>hardware_interface/EffortJointInterface</hardwareInterface>
+      <mechanicalReduction>1</mechanicalReduction>
+    </actuator>
+  </transmission>
+</xacro:macro>
 </robot>

Commit message: controller working! 2 joint gazebo launch

File: arctos_urdf_description/urdf/arctos_urdf.urdf (robot description, URDF)
Before this commit: robot arctos_urdf, 0 links, 0 joints
Links:
- added link world
Joints:
- added joint world_to_base_link: type fixed, parent world, child base_link
