Commit message: temp: TOBE DELETED

File: arctos_urdf_description/urdf/arctos_urdf.xacro (robot description, xacro)
@@ -2,4 +2,5 @@
 <robot name="arctos_urdf" xmlns:xacro="http://www.ros.org/wiki/xacro">
 <xacro:include filename="$(find arctos_urdf_description)/urdf/joint_link.xacro"/>
+<xacro:include filename="$(find arctos_urdf_description)/urdf/arctos_gripper.xacro"/>
 <!-- Start of Selection -->
 <material name="paint_metallic_blue_2">
@@ -71,4 +72,5 @@
     ixx="5.2e-05" iyy="0.000103" izz="5.2e-05" ixy="-0.0" iyz="0.0" ixz="0.0"
 />
+<!-- <xacro:gripper parent="Link_6_1" origin_xyz="0.0 -0.006085 0.0" /> -->
 <xacro:arctos_link
     name="Gripper_1"
@@ -162,10 +164,10 @@
 <xacro:transmission name="joint1_tran" joint_name="joint1" actuator_name="joint1_actr"/>
 <xacro:transmission name="joint2_tran" joint_name="joint2" actuator_name="joint2_actr"/>
+<xacro:transmission name="joint5_tran" joint_name="joint5" actuator_name="joint5_actr"/>
 <xacro:transmission name="joint3_tran" joint_name="joint3" actuator_name="joint3_actr"/>
 <xacro:transmission name="joint4_tran" joint_name="joint4" actuator_name="joint4_actr"/>
-<xacro:transmission name="joint5_tran" joint_name="joint5" actuator_name="joint5_actr"/>
 <xacro:transmission name="joint6_tran" joint_name="joint6" actuator_name="joint6_actr"/>
-<xacro:transmission name="jaw1_tran" joint_name="jaw1" actuator_name="jaw1_actr"/>
-<xacro:transmission name="jaw2_tran" joint_name="jaw2" actuator_name="jaw2_actr"/>
+<xacro:transmission_effort name="jaw1_tran" joint_name="jaw1" actuator_name="jaw1_actr"/>
+<xacro:transmission_effort name="jaw2_tran" joint_name="jaw2" actuator_name="jaw2_actr"/>
 <!-- Gazebo plugin -->
 <gazebo>

File: arctos_urdf_description/urdf/joint_link.xacro (robot description, xacro)
@@ -36,7 +36,4 @@
     <type>transmission_interface/SimpleTransmission</type>
     <joint name="${joint_name}">
-      <!-- Use to be Efforjoint interface for gazebo. So the setup was hardware has EffortJoint interface; Software was JointPosition Interface -->
-      <!-- <hardwareInterface>hardware_interface/EffortJointInterface</hardwareInterface> -->
-      <!-- For MoveIt Use JointPositionInterface as Hardware Interface; software has JointTrajectoryController-->
       <hardwareInterface>hardware_interface/PositionJointInterface</hardwareInterface>
     </joint>
@@ -47,3 +44,15 @@
   </transmission>
 </xacro:macro>
+<xacro:macro name="transmission_effort" params="name joint_name actuator_name">
+  <transmission name="${name}">
+    <type>transmission_interface/SimpleTransmission</type>
+    <joint name="${joint_name}">
+      <hardwareInterface>hardware_interface/EffortJointInterface</hardwareInterface>
+    </joint>
+    <actuator name="${actuator_name}">
+      <hardwareInterface>hardware_interface/EffortJointInterface</hardwareInterface>
+      <mechanicalReduction>1</mechanicalReduction>
+    </actuator>
+  </transmission>
+</xacro:macro>
 </robot>
