Commit message: effort gripper achieved. Successfully Tested in Gazebo

File: arctos_urdf_description/urdf/arctos.xacro (robot description, xacro)
@@ -5,6 +5,8 @@
 <!-- Start of Selection -->
 <material name="paint_metallic_blue_2">
-<!-- <color rgba="0.7764705882352941 0.7764705882352941 0.7764705882352941 1.0"/> -->
   <color rgba="0.0 0.0 1.0 1.0"/> <!-- A solid blue color that works in Gazebo -->
+  <gazebo reference="base_link">
+    <material>Gazebo/Blue</material>
+  </gazebo>
 </material>
 <!-- End of Selection -->
@@ -72,29 +74,6 @@
     ixx="5.2e-05" iyy="0.000103" izz="5.2e-05" ixy="-0.0" iyz="0.0" ixz="0.0"
 />
-<!-- <xacro:gripper parent="Link_6_1" origin_xyz="0.0 -0.006085 0.0" /> -->
-<xacro:arctos_link
-    name="Gripper_1"
-    origin_xyz="-0.000193 0.319847 -0.570316" origin_rpy="0 0 0"
-    material_name="paint_metallic_blue_2"
-    inertia_origin_xyz="0.0036112727264542635 -0.014760653808445767 -0.00103677815369696" inertia_origin_rpy="0 0 0"
-    mass="0.5810486809925093"
-    ixx="0.000385" iyy="0.000495" izz="0.000263" ixy="1e-05" iyz="-2e-06" ixz="3e-06"
-/>
-<xacro:arctos_link
-    name="Left_jaw_1"
-    origin_xyz="-0.007934 0.359845 -0.599867" origin_rpy="0 0 0"
-    material_name="paint_metallic_blue_2"
-    inertia_origin_xyz="-0.011142702480351952 -0.009692440309284511 -0.009385792627785827" inertia_origin_rpy="0 0 0"
-    mass="0.07369602565859415"
-    ixx="1.1e-05" iyy="6e-06" izz="1.4e-05" ixy="2e-06" iyz="-0.0" ixz="-0.0"
-/>
-<xacro:arctos_link
-    name="Right_jaw_1"
-    origin_xyz="-0.007934 0.359845 -0.539867" origin_rpy="0 0 0"
-    material_name="paint_metallic_blue_2"
-    inertia_origin_xyz="-0.008289104952972526 -0.009768535307719373 0.009395511902715814" inertia_origin_rpy="0 0 0"
-    mass="0.07312902168719511"
-    ixx="1.1e-05" iyy="6e-06" izz="1.4e-05" ixy="-1e-06" iyz="0.0" ixz="-1e-06"
-/>
+<!-- Gripper Section -->
+<xacro:gripper parent="Link_6_1" origin_xyz="0.0 -0.006085 0.0" />
 <xacro:arctos_joint
   name="joint1" type="continuous"
@@ -139,26 +118,4 @@
   limit_u="${pi}" limit_l="${-pi}" limit_e="100" limit_v="1"
 />
-<xacro:arctos_joint
-  name="gripper" type="fixed"
-  parent="Link_6_1" child="Gripper_1"
-  origin_xyz="0.0 -0.006085 0.0" origin_rpy="0 0 0"
-  axis_xyz="0 0 0"
-  limit_u="0" limit_l="0" limit_e="0" limit_v="0"
-/>
-<xacro:arctos_joint
-  name="jaw1" type="prismatic"
-  parent="Gripper_1" child="Left_jaw_1"
-  origin_xyz="0.007741 -0.039998 0.029551" origin_rpy="0 0 0"
-  axis_xyz="-0.0 0.0 -1.0"
-  limit_u="0.015" limit_l="0.0" limit_e="100" limit_v="100"
-/>
-<xacro:arctos_joint
-  name="jaw2" type="prismatic"
-  parent="Gripper_1" child="Right_jaw_1"
-  origin_xyz="0.007741 -0.039998 -0.030449" origin_rpy="0 0 0"
-  axis_xyz="0.0 -0.0 1.0"
-  limit_u="0.015" limit_l="0.0" limit_e="100" limit_v="100"
-/>
-<!-- END of Gripper Section -->
 <!-- Transmission section -->
 <xacro:transmission name="joint1_tran" joint_name="joint1" actuator_name="joint1_actr"/>
@@ -168,6 +125,4 @@
 <xacro:transmission name="joint4_tran" joint_name="joint4" actuator_name="joint4_actr"/>
 <xacro:transmission name="joint6_tran" joint_name="joint6" actuator_name="joint6_actr"/>
-<xacro:transmission name="jaw1_tran" joint_name="jaw1" actuator_name="jaw1_actr"/>
-<xacro:transmission name="jaw2_tran" joint_name="jaw2" actuator_name="jaw2_actr"/>
 <!-- Gazebo plugin -->
 <gazebo>

File: arctos_urdf_description/urdf/arctos_gripper.xacro (robot description, xacro)
@@ -4,4 +4,23 @@
 <!-- Arctos Simple Pinch Gripper -->
 <xacro:macro name="gripper" params="parent origin_xyz">
+    <!-- ros control plugin with mimic-->
+    <xacro:macro name="mimic_joint_plugin_gazebo" params="parent_joint mimic_joint has_pid:=false multiplier:=1.0 offset:=0 sensitiveness:=0.0 max_effort:=2000 robot_namespace:='/arctos'">
+        <gazebo>
+            <plugin name="${mimic_joint}_mimic_joint_plugin" filename="libroboticsgroup_gazebo_mimic_joint_plugin.so">
+                <joint>${parent_joint}</joint>
+                <mimicJoint>${mimic_joint}</mimicJoint>
+                <xacro:if value="${has_pid}">
+                    <hasPID />
+                </xacro:if>
+                <multiplier>${multiplier}</multiplier>
+                <offset>${offset}</offset>
+                <sensitiveness>${sensitiveness}</sensitiveness>
+                <maxEffort>${max_effort}</maxEffort>
+                <xacro:unless value="${robot_namespace == ''}">
+                    <robotNamespace>${robot_namespace}</robotNamespace>
+                </xacro:unless>
+            </plugin>
+        </gazebo>
+    </xacro:macro>
     <!-- Gripper Connector -->
     <xacro:arctos_link
@@ -21,4 +40,12 @@
     />
     <!-- Jaw Left -->
+    <joint name="jaw1" type="prismatic">
+        <parent link="Gripper_1"/>
+        <child link="Left_jaw_1"/>
+        <axis xyz="-0.0 0.0 -1.0"/>
+        <limit lower="0.0" upper="0.015" velocity="100" effort="100"/>
+        <origin xyz="0.007741 -0.039998 0.029551" rpy="0 0 0"/>
+        <dynamics damping="1" friction="10"/>
+    </joint>
     <xacro:arctos_link
         name="Left_jaw_1"
@@ -29,14 +56,21 @@
         ixx="1.1e-05" iyy="6e-06" izz="1.4e-05" ixy="2e-06" iyz="-0.0" ixz="-0.0"
     />
-    <!-- <joint name="jaw1" type="prismatic"> -->
-    <joint name="jaw1" type="prismatic">
+    <gazebo reference="Left_jaw_1">
+    <material>Gazebo/Green</material>
+    </gazebo>
+    <xacro:transmission_effort name="left_jaw_tran" joint_name="jaw1" actuator_name="actr_left_jaw"/>
+    <!-- <joint name="jaw2" type="prismatic"> -->
+    <joint name="jaw2" type="prismatic">
         <parent link="Gripper_1"/>
-        <child link="Left_jaw_1"/>
-        <axis xyz="-0.0 0.0 -1.0"/>
-        <limit lower="0.0" upper="0.015" velocity="100" effort="100"/>
-        <origin xyz="0.007741 -0.039998 0.029551" rpy="0 0 0"/>
+        <child link="Right_jaw_1"/>
+        <axis xyz="0.0 -0.0 1.0"/>
+        <limit lower="0.0" upper="0.015" velocity="100" effort="1000"/>
+        <origin xyz="0.007741 -0.039998 -0.030449" rpy="0 0 0"/>
         <dynamics damping="1" friction="10"/>
+        <mimic joint="jaw1" multiplier="1.0" offset="0.0"/>
     </joint>
-    <xacro:transmission_effort name="left_jaw_tran" joint_name="jaw1" actuator_name="actr_left_jaw"/>
+    <!-- <xacro:transmission_effort name="right_jaw_tran" joint_name="jaw2" actuator_name="actr_right_jaw"/> -->
+    <xacro:mimic_joint_plugin_gazebo  parent_joint="jaw1" mimic_joint="jaw2"
+                                        has_pid="false" multiplier="1.0" max_effort="200" />
     <!-- Jaw Right -->
     <xacro:arctos_link
@@ -48,53 +82,4 @@
         ixx="1.1e-05" iyy="6e-06" izz="1.4e-05" ixy="-1e-06" iyz="0.0" ixz="-1e-06"
     />
-    <!-- <joint name="jaw2" type="prismatic"> -->
-    <joint name="jaw2" type="prismatic">
-        <parent link="Gripper_1"/>
-        <child link="Right_jaw_1"/>
-        <axis xyz="0.0 -0.0 1.0"/>
-        <limit lower="0.0" upper="0.015" velocity="100" effort="100"/>
-        <origin xyz="0.007741 -0.039998 -0.030449" rpy="0 0 0"/>
-        <dynamics damping="1" friction="10"/>
-        <mimic joint="jaw1" multiplier="-1.0" offset="0.0"/>
-    </joint>
-    <xacro:transmission_effort name="right_jaw_tran" joint_name="jaw2" actuator_name="actr_right_jaw"/>
-    <!-- ros control plugin with mimic-->
-    <xacro:macro name="mimic_joint_plugin_gazebo" params="parent_joint mimic_joint has_pid:=false multiplier:=-1.0 offset:=0 sensitiveness:=0.0 max_effort:=200 robot_namespace:='/arctos'">
-        <gazebo>
-            <plugin name="${mimic_joint}_mimic_joint_plugin" filename="libroboticsgroup_upatras_gazebo_mimic_joint_plugin.so">
-                <joint>${parent_joint}</joint>
-                <mimicJoint>${mimic_joint}</mimicJoint>
-                <xacro:if value="${has_pid}">
-                    <hasPID />
-                </xacro:if>
-                <multiplier>${multiplier}</multiplier>
-                <offset>${offset}</offset>
-                <sensitiveness>${sensitiveness}</sensitiveness>
-                <maxEffort>${max_effort}</maxEffort>
-                <xacro:unless value="${robot_namespace == '/cobot'}">
-                    <robotNamespace>${robot_namespace}</robotNamespace>
-                </xacro:unless>
-            </plugin>
-        </gazebo>
-    </xacro:macro>
-    <xacro:mimic_joint_plugin_gazebo  parent_joint="jaw1" mimic_joint="jaw2"
-                                        has_pid="false" multiplier="-1.0" max_effort="200" />
-    <gazebo>
-        <plugin name="gazebo_grasp_fix" filename="libgazebo_grasp_fix.so">
-            <arm>
-                <arm_name>gripper</arm_name>
-                <palm_link>Gripper_1</palm_link>
-                <gripper_link>Right_jaw_1</gripper_link>
-                <gripper_link>Left_jaw_1</gripper_link>
-            </arm>
-            <forces_angle_tolerance>100</forces_angle_tolerance>
-            <update_rate>10</update_rate>
-            <grip_count_threshold>4</grip_count_threshold>
-            <max_grip_count>10</max_grip_count>
-            <release_tolerance>0.005</release_tolerance>
-            <disable_collision_on_attach>false</disable_collision_on_attach>
-            <contact_topic>__default_topic__</contact_topic>
-        </plugin>
-    </gazebo>
 </xacro:macro>
 </robot>
